Commit message: Add files via upload

File: turtlebot3_description/urdf/turtlebot3_burger.urdf.xacro (robot description, xacro)
@@ -1,4 +1,4 @@
 <?xml version="1.0" ?>
-<robot name="turtlebot3_burger" xmlns:xacro="http://ros.org/wiki/xacro">
+<robot name="turtlebot3" xmlns:xacro="http://ros.org/wiki/xacro">
   <xacro:include filename="$(find turtlebot3_description)/urdf/common_properties.xacro"/>
   <link name="base_footprint"/>
@@ -18,7 +18,7 @@
     </inertial>
     <visual>
-      <origin xyz="0 0.076 0" rpy="0 0 0" />
+      <origin xyz="0 0.076 0" rpy="1.5708 0 0" />
       <geometry>
-        <mesh filename="package://turtlebot3_burger/meshes/base_link.STL" />
+        <mesh filename="package://turtlebot3_description/meshes/bases/base_link.STL" />
       </geometry>
       <material name="">
@@ -29,5 +29,5 @@
       <origin xyz="0 0 0" rpy="0 0 0" />
       <geometry>
-        <mesh filename="package://turtlebot3_burger/meshes/base_link.STL" />
+        <mesh filename="package://turtlebot3_description/meshes/bases/base_link.STL" />
       </geometry>
     </collision>
@@ -45,5 +45,5 @@
       <origin xyz="0 0 0" rpy="0 0 0" />
       <geometry>
-        <mesh filename="package://turtlebot3_burger/meshes/wheel_left_link.STL" />
+        <mesh filename="package://turtlebot3_description/meshes/wheels/wheel_left_link.STL" />
       </geometry>
       <material name="">
@@ -54,5 +54,5 @@
       <origin xyz="0 0 0" rpy="0 0 0" />
       <geometry>
-        <mesh filename="package://turtlebot3_burger/meshes/wheel_left_link.STL" />
+        <mesh filename="package://turtlebot3_description/meshes/wheels/wheel_left_link.STL" />
       </geometry>
     </collision>
@@ -78,5 +78,5 @@
       <origin xyz="0 0 0" rpy="0 0 0" />
       <geometry>
-        <mesh filename="package://turtlebot3_burger/meshes/wheel_right_link.STL" />
+        <mesh filename="package://turtlebot3_description/meshes/wheels/wheel_right_link.STL" />
       </geometry>
       <material name="">
@@ -87,5 +87,5 @@
       <origin xyz="0 0 0" rpy="0 0 0" />
       <geometry>
-        <mesh filename="package://turtlebot3_burger/meshes/wheel_right_link.STL" />
+        <mesh filename="package://turtlebot3_description/meshes/wheels/wheel_right_link.STL" />
       </geometry>
     </collision>
@@ -111,5 +111,5 @@
       <origin xyz="0 0 0" rpy="0 0 0" />
       <geometry>
-        <mesh filename="package://turtlebot3_burger/meshes/base_scan.STL" />
+        <mesh filename="package://turtlebot3_description/meshes/bases/base_scan.STL" />
       </geometry>
       <material name="">
@@ -120,5 +120,5 @@
       <origin xyz="0 0 0" rpy="0 0 0" />
       <geometry>
-        <mesh filename="package://turtlebot3_burger/meshes/base_scan.STL" />
+        <mesh filename="package://turtlebot3_description/meshes/bases/base_scan.STL" />
       </geometry>
     </collision>
